File: schematic_ap.sch (EAGLE design)
At the start: 51 parts, among them J1 FTDI_DEVICE, M1 WIRELESS-NRF24L01, U1 ATMEGA328P_TQFP, U3 MPU-6050

Commit message: Post-Design Changes
Changes according to recommendations
Parts:
- removed C_CP1: 1miF, rcl:C-USC0603
- removed C_CP2, C_CP3: 2.2miF, rcl:C-USC0603
- removed C_G1, C_G4, C_R: 100 nF, rcl:C-USC0603
- removed C_G2: 10 nF, rcl:C-USC0603
- removed C_G3: 2.2 nF, rcl:C-USC0603
- removed D1, D2: RED, LEDs:LED-RED0603
- removed D3, D4: GREEN, LEDs:LED-GREEN0603
- removed R_LED1, R_LED2, R_LED3, R_LED4: 150 Ω, resistor:R-US_R0603
- removed R_M1, R_M2, R_M3, R_M4: 10 kΩ, resistor:R-US_R0603
- removed R_VD1: 100 kΩ, resistor:R-US_R0603
- removed U$1, U$2, U$6, U$8: 2N7002P, 2N7002P:2N7002P
- removed U3: MPU-6050, MPU-6050:MPU-6050
- added C1CP: 1 uF, rcl:C-USC0603
- added C2CP, C3CP: 2.2 uF, rcl:C-USC0603
- added CRES: 100 nF, rcl:C-USC0603
- added D1LED, D2LED: RED, LEDs:LED-RED0603
- added D3LED, D4LED: GREEN, LEDs:LED-GREEN0603
- added R1LED, R2LED, R3LED, R4LED: 150 Ω, resistor:R-US_R0603
- added R1VD, RM1, RM2, RM3, RM4: 10 kΩ, resistor:R-US_R0603
- added U2: GY-521MPU6050, quad:GY-521MPU6050
- added U4, U5, U6, U7: STN4NF03L, STN4NF03L:STN4NF03L
- C1RF: value 100 miF -> 10 uF
- CBAT: value 100 miF -> 100 uF
- R2VD: value 100 kΩ -> 10 kΩ
- R5: value 7 kΩ -> 10 kΩ
- renumbered C_BAT to CBAT, C_DEC1 to C1DEC, C_DEC2 to C2DEC, C_DEC3 to C3DEC, C_OSC1 to C1OSC, C_OSC2 to C2OSC, C_RF1 to C1RF, C_RF2 to C2RF, D_M1 to DM1, D_M2 to DM2, D_M3 to DM3, D_M4 to DM4, R_VD2 to R2VD
Connections:
- net RX/TX renamed RX
- net TX/RX renamed TX
- removed net AVCC: C2DEC.1, U1.AVCC
- removed net B_OUT: CBAT.1, C_CP2.1, DM1.GPIN, DM2.GPIN, DM3.GPIN, DM4.GPIN, R2VD.2, U$11.+, U$3.EN, U$3.VIN, U$4.+, U$5.+, U$7.+, U$9.+
- removed net D_OUT1: D1.A, U1.PB0(ICP)
- removed net D_OUT2: D2.A, U1.PC0(ADC0)
- removed net D_OUT3: D3.A, U1.PC1(ADC1)
- removed net D_OUT4: D4.A, U1.PD2(INT0)
- removed net N$11: R_M1.2, U$2.S
- removed net N$18: R_M2.2, U$1.S
- removed net N$22: R_M3.2, U$6.S
- removed net N$25: R_M4.2, U$8.S
- removed net N$5: C_G3.1, U3.CPOUT
- removed net N$6: C_G4.1, U3.REGOUT
- removed net N$7: R2VD.1, R_VD1.2
- removed net P_OUT: C1OSC.1, C1RF.1, C2OSC.1, C2RF.1, C3DEC.1, C_CP3.1, C_G1.1, C_G2.1, J1.VCC, M1.VCC, R5.1, U$3.VOUT, U1.VCC@4, U1.VCC@6, U3.VDD, U3.VLOGIC
- new net 3V3: C1OSC.1, C1RF.1, C2DEC.1, C2OSC.1, C2RF.1, C3CP.1, C3DEC.1, J1.VCC, M1.VCC, R5.1, U$3.VOUT, U1.AVCC, U1.VCC@4, U1.VCC@6, U2.VCC
- new net INT: U1.PD4(XCK/T0), U2.INT
- new net LED1: D1LED.A, U1.PB0(ICP)
- new net LED2: D2LED.A, U1.PC0(ADC0)
- new net LED3: D3LED.A, U1.PC1(ADC1)
- new net LED4: D4LED.A, U1.PD2(INT0)
- new net VBAT: C2CP.1, CBAT.1, DM1.GPIN, DM2.GPIN, DM3.GPIN, DM4.GPIN, R2VD.2, U$11.+, U$3.EN, U$3.VIN, U$4.+, U$5.+, U$7.+, U$9.+
- new net VDIV: R1VD.2, R2VD.1, U1.PC2(ADC2)
- net GND: now also C2CP.2, C3CP.2, R1LED.1, R1VD.1, R2LED.1, R3LED.1, R4LED.1, RM1.1, RM2.1, RM3.1, RM4.1, U1.AGND, U1.GND@3, U1.GND@5, U2.GND, U4.3, U5.3, U6.3, U7.3; no longer C_CP2.2, C_CP3.2, C_G1.2, C_G2.2, C_G3.2, C_G4.2, R_LED1.1, R_LED2.1, R_LED3.1, R_LED4.1, R_M1.1, R_M2.1, R_M3.1, R_M4.1, R_VD1.1, U3.GND
- net N$12: now also C1CP.1; no longer C_CP1.1
- net N$13: now also C1CP.2; no longer C_CP1.2
- net N$15: now also U7.2; no longer U$2.D
- net N$19: now also D4LED.C, R4LED.2; no longer D4.C, R_LED4.2
- net N$20: now also U6.2; no longer U$1.D
- net N$21: now also D2LED.C, R2LED.2; no longer D2.C, R_LED2.2
- net N$23: now also D3LED.C, R3LED.2; no longer D3.C, R_LED3.2
- net N$24: now also U5.2; no longer U$6.D
- net N$26: now also U4.2; no longer U$8.D
- net N$3: now also CRES.1; no longer C_R.1
- net N$30: now also D1LED.C, R1LED.2; no longer D1.C, R_LED1.2
- net PWM1: now also RM1.2, U7.1; no longer U$2.G
- net PWM2: now also RM2.2, U6.1; no longer U$1.G
- net PWM3: now also RM3.2, U5.1; no longer U$6.G
- net PWM4: now also RM4.2, U4.1; no longer U$8.G
- net RESET: now also CRES.2; no longer C_R.2
- net SCL: now also U2.SCL; no longer U3.SCL
- net SDA: now also U2.SDA; no longer U3.SDA
Other:
- moved on the sheet: J1, R5, U$10, U$3
