File: schematic_ap_team10.brd (EAGLE design)
At the start: 47 x 28 mm, 47 parts, among them J1 FTDI_DEVICE, M1 WIRELESS-NRF24L01, U1 ATMEGA328P_TQFP, U2 GY-521MPU6050

Commit message: LED Resistor Update
150Ohm -> 65Ohm
Parts:
- R1LED, R2LED, R3LED, R4LED: value 150 Ω -> 65 Ω
Changed lines of the file:
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@@
 <layer number="14" name="Route14" color="1" fill="6" visible="no" active="no"/>
 <layer number="15" name="Route15" color="4" fill="6" visible="no" active="no"/>
-<layer number="16" name="Bottom" color="1" fill="1" visible="yes" active="yes"/>
+<layer number="16" name="Bottom" color="1" fill="1" visible="no" active="yes"/>
 <layer number="17" name="Pads" color="2" fill="1" visible="yes" active="yes"/>
 <layer number="18" name="Vias" color="2" fill="1" visible="yes" active="yes"/>
 <layer number="19" name="Unrouted" color="6" fill="1" visible="yes" active="yes"/>
 <layer number="20" name="Dimension" color="24" fill="1" visible="yes" active="yes"/>
-<layer number="21" name="tPlace" color="7" fill="1" visible="no" active="yes"/>
+<layer number="21" name="tPlace" color="7" fill="1" visible="yes" active="yes"/>
 <layer number="22" name="bPlace" color="7" fill="1" visible="yes" active="yes"/>
-<layer number="23" name="tOrigins" color="15" fill="1" visible="no" active="yes"/>
+<layer number="23" name="tOrigins" color="15" fill="1" visible="yes" active="yes"/>
 <layer number="24" name="bOrigins" color="15" fill="1" visible="yes" active="yes"/>
-<layer number="25" name="tNames" color="7" fill="1" visible="no" active="yes"/>
+<layer number="25" name="tNames" color="7" fill="1" visible="yes" active="yes"/>
 <layer number="26" name="bNames" color="7" fill="1" visible="yes" active="yes"/>
 <layer number="27" name="tValues" color="7" fill="1" visible="no" active="yes"/>
@@
 <element name="J1" library="quad" package="FTDI_DEVICE_SIDE" value="FTDI_DEVICE" x="34.671" y="26.035" smashed="yes" rot="R180"/>
 <element name="M1" library="quad" package="WIRELESS-NRF24L01" value="WIRELESS-NRF24L01" x="32.385" y="16.51" smashed="yes" rot="R180"/>
-<element name="R1LED" library="resistor" package="R0603" value="150 Ω" x="6.35" y="2.032" smashed="yes" rot="MR180">
-<attribute name="VALUE" x="5.207" y="1.397" size="0.6096" layer="28" rot="MR180"/>
+<element name="R1LED" library="resistor" package="R0603" value="65 Ω" x="6.35" y="2.032" smashed="yes" rot="MR180">
+<attribute name="VALUE" x="5.461" y="1.397" size="0.6096" layer="28" rot="MR180"/>
 </element>
 <element name="R1VD" library="resistor" package="R0603" value="10 kΩ" x="14.732" y="6.35" smashed="yes" rot="R90">
 <attribute name="VALUE" x="16.002" y="5.207" size="0.6096" layer="27" rot="R90"/>
 </element>
-<element name="R2LED" library="resistor" package="R0603" value="150 Ω" x="44.069" y="4.064" smashed="yes" rot="MR180">
-<attribute name="VALUE" x="42.926" y="3.429" size="0.6096" layer="28" rot="MR180"/>
+<element name="R2LED" library="resistor" package="R0603" value="65 Ω" x="44.069" y="4.064" smashed="yes" rot="MR180">
+<attribute name="VALUE" x="43.18" y="3.429" size="0.6096" layer="28" rot="MR180"/>
 </element>
 <element name="R2VD" library="resistor" package="R0603" value="10 kΩ" x="9.525" y="6.604" smashed="yes" rot="R270">
 <attribute name="VALUE" x="8.89" y="5.461" size="0.6096" layer="27" rot="R90"/>
 </element>
-<element name="R3LED" library="resistor" package="R0603" value="150 Ω" x="44.069" y="24.13" smashed="yes" rot="MR180">
-<attribute name="VALUE" x="42.926" y="25.4" size="0.6096" layer="28" rot="MR180"/>
-</element>
-<element name="R4LED" library="resistor" package="R0603" value="150 Ω" x="6.35" y="26.035" smashed="yes" rot="MR0">
+<element name="R3LED" library="resistor" package="R0603" value="65 Ω" x="44.069" y="24.13" smashed="yes" rot="MR180">
+<attribute name="VALUE" x="43.18" y="25.4" size="0.6096" layer="28" rot="MR180"/>
+</element>
+<element name="R4LED" library="resistor" package="R0603" value="65 Ω" x="6.35" y="26.035" smashed="yes" rot="MR0">
 <attribute name="VALUE" x="7.366" y="26.67" size="0.6096" layer="28" rot="MR0"/>
 </element>
